File: pcb/main_v2/main_v2.kicad_pcb (KiCad board)
At the start: 2 copper layers, 79.4 x 53.3 mm, 24 parts, among them J1 AS5600, J2 Btn, Q1 DMN3051L, SW1 SW_Push, SW2 SW_Push, U2 24AA02-OT, U3 PCA9536D

Commit message: PCB - small board
Parts:
- added J3: Btn, Connector_PinHeader_2.54mm:PinHeader_1x02_P2.54mm_Vertical, F.Cu at (131.2, 119.7)
- added SW3: SW_Push, Button_Switch_THT:SW_PUSH_6mm_H7.3mm, F.Cu at (115.6, 117.5)
Routing:
- net Net-(J3-Pin_2): track 0.00 -> 15.0 mm
- net Net-(J3-Pin_1): track 0.00 -> 6.50 mm
Other:
- board size 79.4 x 53.3 mm -> 79.4 x 72.9 mm
